Commit message: Add full-body 3D control with live slider-to-preview sync
- Add arms, hands, and legs control via BodyPage and expanded control panel

- Wire sliders directly to URDF joints through robotLiveController

- Compile full InMoov URDF with official meshes, generated legs, and white PLA materials

- Add bodyStore, joint mapping, gallery poses, and full-body Arduino firmware

- Update Flask routes, run.bat pipeline, and gitignore for build/vendor artifacts

File: models/inmoov/inmoov.urdf (robot description, URDF)
Before this commit: robot inmoov, 34 links, 33 joints
Links:
- added link kinect2_link; visual mesh filename=package://inmoov_meshes/meshes/kinectone.stl scale=0.001 0.001 0.001
- added link l_foot_link
- added link l_foot_roll_link; visual box size=0.18 0.08 0.04
- added link l_hip_link; visual sphere radius=0.04
- added link l_index_link; visual box size=0.07 0.01 0.01
- added link l_middle_link; visual box size=0.075 0.01 0.01
- added link l_pinky_link; visual box size=0.065 0.01 0.01
- added link l_ring_link; visual box size=0.07 0.01 0.01
- added link l_shin_link; visual cylinder length=0.32 radius=0.03
- added link l_thigh_link; visual cylinder length=0.36 radius=0.035
- added link l_thumb_link; visual box size=0.05 0.012 0.012
- added link r_foot_link
- added link r_foot_roll_link; visual box size=0.18 0.08 0.04
- added link r_hip_link; visual sphere radius=0.04
- added link r_index_link; visual box size=0.07 0.01 0.01
- added link r_middle_link; visual box size=0.075 0.01 0.01
- added link r_pinky_link; visual box size=0.065 0.01 0.01
- added link r_ring_link; visual box size=0.07 0.01 0.01
- added link r_shin_link; visual cylinder length=0.32 radius=0.03
- added link r_thigh_link; visual cylinder length=0.36 radius=0.035
- added link r_thumb_link; visual box size=0.05 0.012 0.012
Joints:
- added joint kinect2_joint: type fixed, parent torso_link, child kinect2_link, origin xyz=0 0 0.066 rpy=-1.57 0 -1.57
- added joint l_ankle_joint: type revolute, parent l_shin_link, child l_foot_link, origin xyz=0 0 -0.32 rpy=0 0 0, axis 1 0 0, limit lower=-0.8 upper=0.8 effort=1000 velocity=1
- added joint l_foot_roll_joint: type revolute, parent l_foot_link, child l_foot_roll_link, origin xyz=0 0 0 rpy=0 0 0, axis 0 0 1, limit lower=-0.5 upper=0.5 effort=100 velocity=1
- added joint l_hip_lift_joint: type revolute, parent l_hip_link, child l_thigh_link, origin xyz=0 0 0 rpy=0 0 0, axis 1 0 0, limit lower=-1.2 upper=1.2 effort=1000 velocity=1
- added joint l_hip_pan_joint: type revolute, parent mid_stomach_link, child l_hip_link, origin xyz=0 0.09 1.02 rpy=0 0 0, axis 0 0 1, limit lower=-0.8 upper=0.8 effort=1000 velocity=1
- added joint l_index_joint: type revolute, parent l_hand_link, child l_index_link, origin xyz=0.02 -0.01 0 rpy=0 0 0, axis 0 1 0, limit lower=0 upper=1.4 effort=100 velocity=1
- added joint l_knee_joint: type revolute, parent l_thigh_link, child l_shin_link, origin xyz=0 0 -0.36 rpy=0 0 0, axis 1 0 0, limit lower=0 upper=2.2 effort=1000 velocity=1
- added joint l_middle_joint: type revolute, parent l_hand_link, child l_middle_link, origin xyz=0.02 0 0 rpy=0 0 0, axis 0 1 0, limit lower=0 upper=1.4 effort=100 velocity=1
- added joint l_pinky_joint: type revolute, parent l_hand_link, child l_pinky_link, origin xyz=0.02 0.02 0 rpy=0 0 0, axis 0 1 0, limit lower=0 upper=1.4 effort=100 velocity=1
- added joint l_ring_joint: type revolute, parent l_hand_link, child l_ring_link, origin xyz=0.02 0.01 0 rpy=0 0 0, axis 0 1 0, limit lower=0 upper=1.4 effort=100 velocity=1
- added joint l_thumb_joint: type revolute, parent l_hand_link, child l_thumb_link, origin xyz=0.02 -0.03 0 rpy=0 0 0, axis 0 1 0, limit lower=0 upper=1.2 effort=100 velocity=1
- added joint r_ankle_joint: type revolute, parent r_shin_link, child r_foot_link, origin xyz=0 0 -0.32 rpy=0 0 0, axis 1 0 0, limit lower=-0.8 upper=0.8 effort=1000 velocity=1
- added joint r_foot_roll_joint: type revolute, parent r_foot_link, child r_foot_roll_link, origin xyz=0 0 0 rpy=0 0 0, axis 0 0 1, limit lower=-0.5 upper=0.5 effort=100 velocity=1
- added joint r_hip_lift_joint: type revolute, parent r_hip_link, child r_thigh_link, origin xyz=0 0 0 rpy=0 0 0, axis 1 0 0, limit lower=-1.2 upper=1.2 effort=1000 velocity=1
- added joint r_hip_pan_joint: type revolute, parent mid_stomach_link, child r_hip_link, origin xyz=0 -0.09 1.02 rpy=0 0 0, axis 0 0 1, limit lower=-0.8 upper=0.8 effort=1000 velocity=1
- added joint r_index_joint: type revolute, parent r_hand_link, child r_index_link, origin xyz=0.02 0.01 0 rpy=0 0 0, axis 0 1 0, limit lower=0 upper=1.4 effort=100 velocity=1
- added joint r_knee_joint: type revolute, parent r_thigh_link, child r_shin_link, origin xyz=0 0 -0.36 rpy=0 0 0, axis 1 0 0, limit lower=0 upper=2.2 effort=1000 velocity=1
- added joint r_middle_joint: type revolute, parent r_hand_link, child r_middle_link, origin xyz=0.02 0 0 rpy=0 0 0, axis 0 1 0, limit lower=0 upper=1.4 effort=100 velocity=1
- added joint r_pinky_joint: type revolute, parent r_hand_link, child r_pinky_link, origin xyz=0.02 -0.02 0 rpy=0 0 0, axis 0 1 0, limit lower=0 upper=1.4 effort=100 velocity=1
- added joint r_ring_joint: type revolute, parent r_hand_link, child r_ring_link, origin xyz=0.02 -0.01 0 rpy=0 0 0, axis 0 1 0, limit lower=0 upper=1.4 effort=100 velocity=1
- added joint r_thumb_joint: type revolute, parent r_hand_link, child r_thumb_link, origin xyz=0.02 0.03 0 rpy=0 0 0, axis 0 1 0, limit lower=0 upper=1.2 effort=100 velocity=1
- joint l_elbow_flex_joint: axis (none) -> 0 1 0; limit (none) -> lower=-1.484 upper=-0.262 effort=1000 velocity=1; type fixed -> revolute
- joint l_shoulder_lift_joint: axis (none) -> 0 1 0; limit (none) -> lower=-2.356 upper=0.785 effort=1000 velocity=1; type fixed -> revolute
- joint l_shoulder_out_joint: axis (none) -> 1 0 0; limit (none) -> lower=0.087 upper=1.047 effort=1000 velocity=1; type fixed -> revolute
- joint l_upper_arm_roll_joint: axis (none) -> 0 0 1; limit (none) -> lower=-1.57 upper=1.57 effort=1000 velocity=1; type fixed -> revolute
- joint l_wrist_roll_joint: axis (none) -> 0 0 1; limit (none) -> lower=-1.57 upper=1.57 effort=1000 velocity=1; type fixed -> revolute
- joint r_elbow_flex_joint: axis (none) -> 0 1 0; limit (none) -> lower=-1.484 upper=-0.262 effort=1000 velocity=1; type fixed -> revolute
- joint r_shoulder_lift_joint: axis (none) -> 0 1 0; limit (none) -> lower=-2.356 upper=0.785 effort=1000 velocity=1; type fixed -> revolute
- joint r_shoulder_out_joint: axis (none) -> 1 0 0; limit (none) -> lower=-1.047 upper=-0.087 effort=1000 velocity=1; type fixed -> revolute
- joint r_upper_arm_roll_joint: axis (none) -> 0 0 1; limit (none) -> lower=-1.57 upper=1.57 effort=1000 velocity=1; type fixed -> revolute
- joint r_wrist_roll_joint: axis (none) -> 0 0 1; limit (none) -> lower=-1.57 upper=1.57 effort=1000 velocity=1; type fixed -> revolute
- joint waist_roll_joint: axis (none) -> 1 0 0; limit (none) -> lower=-0.262 upper=0.262 effort=1000 velocity=1; type fixed -> revolute
